File: ESP32 S3 LM 2 LITE.kicad_pcb (KiCad board)
At the start: 2 copper layers, 25.4 x 69.8 mm, 40 parts, among them J1 Conn_01x22_Pin, J2 USB_C_Receptacle_USB2.0_16P, J3 USB_C_Receptacle_USB2.0_16P, J4 Conn_01x22_Pin, Q1 SS8050, Q2 SS8050, SW1 SW_Push, SW2 SW_Push, U1 ESP32-S3-WROOM-1, U2 AMS1117-3.3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

Commit message: Add files via upload
A UPDATED VERIOSN FINISHED NOT REVIEW BY OTHER YET
Parts:
- added R12: 0, Resistor_SMD:R_0603_1608Metric, F.Cu at (108.6, 85.1)
- U1: footprint RF_Module:ESP32-S3-WROOM-1 -> PCM_Espressif:ESP32-S3-WROOM-1
- moved J1 3.20 mm to (89.5, 62.2)
- moved J4 3.20 mm to (112.4, 62.2)
- moved U1 2.89 mm to (101.0, 71.0)
- moved C3 2.83 mm to (102.9, 92.4)
- moved C1 2.82 mm to (94.0, 85.1)
- moved C2 2.82 mm to (108.0, 92.4)
- moved C4 2.82 mm to (95.9, 85.1)
- moved C8 2.82 mm to (95.9, 92.3)
- moved D2 2.82 mm to (95.6, 114.2)
- moved D3 2.82 mm to (95.9, 96.1)
- moved D5 2.82 mm to (109.1, 114.2)
- moved D6 2.82 mm to (97.2, 114.2)
- moved Q1 2.82 mm to (102.9, 95.6)
- moved Q2 2.82 mm to (108.0, 95.6)
- moved R10 2.82 mm to (94.1, 114.2)
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Connections:
- Q1 pad 3: Net-(Q1-C) -> EN
- U1 pad 27: G0 -> Net-(U1-IO0)
Routing:
- net GND: track 18.4 -> 41.1 mm, vias 63 -> 61
- net G0: track 53.0 -> 41.5 mm
- net VBUS: track 25.0 -> 31.5 mm
- net Net-(U1-IO0): track 0.00 -> 5.54 mm
- net DTR: track 28.9 -> 25.6 mm
- net EN: track 81.9 -> 79.3 mm
- net +3.3V: track 128.9 -> 127.4 mm
- net Net-(D5-A): track 12.6 -> 11.6 mm
- net G2: track 13.5 -> 12.5 mm
- net Net-(J2-CC2): track 14.7 -> 13.7 mm
- net G7: track 13.7 -> 12.9 mm
- net /NATIVE_USB_D+: track 68.7 -> 69.4 mm
- net U0TXD: track 64.2 -> 64.8 mm
- net /COM_USB_D+: track 30.4 -> 29.8 mm
- net /COM_USB_D-: track 31.9 -> 31.3 mm
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Other:
- outline, holes or cut-outs redrawn
- board text added: "3.3 V"
- board text added: "41"
- board text added: "BOOT"
- board text added: "CH343G"
- board text added: "COM"
- board text added: "EN"
- board text added: "EPS32 S3 NXRX"
- board text added: "G"
- board text added: "LDO"
- board text added: "NEO"
- board text added: "PWR"
- board text added: "REST"
- board text added: "RX"
- board text added: "TX"
- board text added: "USB"
- board text added: "thsi is logic meso"
