File: ESP32 S3 LM 2 LITE.kicad_sch (KiCad schematic)
At the start: 39 parts, among them J1 Conn_01x22_Pin, J2 USB_C_Receptacle_USB2.0_16P, J3 USB_C_Receptacle_USB2.0_16P, J4 Conn_01x22_Pin, Q1 SS8050, Q2 SS8050, SW1 SW_Push, SW2 SW_Push, U1 ESP32-S3-WROOM-1, U2 AMS1117-3.3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

Commit message: Add files via upload
A UPDATED VERIOSN FINISHED NOT REVIEW BY OTHER YET
Parts:
- added R12: 0, Resistor_SMD:R_0603_1608Metric, symbol Device:R
- U1: footprint RF_Module:ESP32-S3-WROOM-1 -> PCM_Espressif:ESP32-S3-WROOM-1
- U2: value AMS1117-3.3 -> TL1117-3.3
Connections:
- net G0: now also R12.2; no longer U1.27 (IO0)
- new net: R12.1, U1.27 (IO0)
Other:
- note added: "COM PORT"
- note added: "LDO"
- note added: "USB PORT"
- moved on the sheet: C1, C2, C3, C4, C5, C6, D1, R8, SW1, SW2, U1, U2
